Commit message: Fix small example issues

File: examples/piper/piper_left.urdf (robot description, URDF)
Before this commit: robot piper_description, 9 links, 8 joints
Links:
- link base_link: geometry collision mesh filename=base_link.STL; visual mesh filename=base_link.STL
- link link1: geometry collision mesh filename=link1.STL; visual mesh filename=link1.STL
- link link2: geometry collision mesh filename=link2.STL; visual mesh filename=link2.STL
- link link3: geometry collision mesh filename=link3.STL; visual mesh filename=link3.STL
- link link4: geometry collision mesh filename=link4.STL; visual mesh filename=link4.STL
- link link5: geometry collision mesh filename=link5.STL; visual mesh filename=link5.STL
- link link6: geometry collision mesh filename=link6.STL; visual mesh filename=link6.STL
- link link7: geometry collision mesh filename=link7.STL; visual mesh filename=link7.STL
- link link8: geometry collision mesh filename=link8.STL; visual mesh filename=link8.STL

File: examples/piper/piper_left_pred.urdf (robot description, URDF)
Before this commit: robot piper_description, 9 links, 8 joints
Links:
- link base_link: geometry collision mesh filename=base_link.STL; visual mesh filename=base_link.STL
- link link1: geometry collision mesh filename=link1.STL; visual mesh filename=link1.STL
- link link2: geometry collision mesh filename=link2.STL; visual mesh filename=link2.STL
- link link3: geometry collision mesh filename=link3.STL; visual mesh filename=link3.STL
- link link4: geometry collision mesh filename=link4.STL; visual mesh filename=link4.STL
- link link5: geometry collision mesh filename=link5.STL; visual mesh filename=link5.STL
- link link6: geometry collision mesh filename=link6.STL; visual mesh filename=link6.STL
- link link7: geometry collision mesh filename=link7.STL; visual mesh filename=link7.STL
- link link8: geometry collision mesh filename=link8.STL; visual mesh filename=link8.STL

File: examples/piper/piper_right.urdf (robot description, URDF)
Before this commit: robot piper_description, 9 links, 8 joints
Links:
- link base_link: geometry collision mesh filename=base_link.STL; visual mesh filename=base_link.STL
- link link1: geometry collision mesh filename=link1.STL; visual mesh filename=link1.STL
- link link2: geometry collision mesh filename=link2.STL; visual mesh filename=link2.STL
- link link3: geometry collision mesh filename=link3.STL; visual mesh filename=link3.STL
- link link4: geometry collision mesh filename=link4.STL; visual mesh filename=link4.STL
- link link5: geometry collision mesh filename=link5.STL; visual mesh filename=link5.STL
- link link6: geometry collision mesh filename=link6.STL; visual mesh filename=link6.STL
- link link7: geometry collision mesh filename=link7.STL; visual mesh filename=link7.STL
- link link8: geometry collision mesh filename=link8.STL; visual mesh filename=link8.STL

File: examples/piper/piper_right_pred.urdf (robot description, URDF)
Before this commit: robot piper_description, 9 links, 8 joints
Links:
- link base_link: geometry collision mesh filename=base_link.STL; visual mesh filename=base_link.STL
- link link1: geometry collision mesh filename=link1.STL; visual mesh filename=link1.STL
- link link2: geometry collision mesh filename=link2.STL; visual mesh filename=link2.STL
- link link3: geometry collision mesh filename=link3.STL; visual mesh filename=link3.STL
- link link4: geometry collision mesh filename=link4.STL; visual mesh filename=link4.STL
- link link5: geometry collision mesh filename=link5.STL; visual mesh filename=link5.STL
- link link6: geometry collision mesh filename=link6.STL; visual mesh filename=link6.STL
- link link7: geometry collision mesh filename=link7.STL; visual mesh filename=link7.STL
- link link8: geometry collision mesh filename=link8.STL; visual mesh filename=link8.STL
