Commit message: Use fixed urdf to do ik

File: examples/so100-remote/so100.urdf (robot description, URDF)
Before this commit: robot SO_5DOF_ARM100_8j_URDF.SLDASM, 7 links, 6 joints
Joints:
- joint Rotation: axis 0 -1 0 -> 0 1 0

File: examples/so100-remote/so100_2.urdf (robot description, URDF)
Before this commit: robot SO_5DOF_ARM100_8j_URDF.SLDASM, 7 links, 6 joints
Links:
- removed link Base
- added link base_link, mass 0.193184127927598; collision mesh filename=Base.STL; visual mesh filename=Base.STL
Joints:
- joint Jaw: origin xyz=-0.0202 -0.0244 0 rpy=3.1416 0 3.1416 -> xyz=-0.0202 -0.0244 0 rpy=0 0 0
- joint Rotation: axis 0 1 0 -> 0 -1 0; parent Base -> base_link
- joint Wrist_Pitch: origin xyz=0 0.0052 0.1349 rpy=0 0 0 -> xyz=0 0.0052 0.1349 rpy=-1.57 0 0
- joint Wrist_Roll: origin xyz=0 -0.0601 0 rpy=0 0 0 -> xyz=0 -0.0601 0 rpy=0 1.57 0

Commit message: Fix CI/CD And improve example

File: examples/so100-remote/so100.urdf (robot description, URDF)
Before this commit: robot SO_5DOF_ARM100_8j_URDF.SLDASM, 7 links, 6 joints
Links:
- link Fixed_Jaw: geometry collision mesh filename=Wrist_Roll_Follower_SO101.STL; visual mesh filename=Fixed_Jaw.STL
- link Moving Jaw: geometry collision mesh filename=Moving_Jaw_SO101.STL; visual mesh filename=Moving Jaw.STL
Joints:
- joint Elbow: limit lower=-0.2 upper=3.14159 effort=0 velocity=0 -> (none); origin xyz=0 0.11257 0.028 rpy=-1.5708 0 0 -> xyz=0 0.11257 0.028 rpy=-0.1 0 0
- joint Jaw: limit lower=0 upper=1.7 effort=0 velocity=0 -> (none)
- joint Pitch: axis -1 0 0 -> 1 0 0; limit lower=-0.1 upper=3.45 effort=0 velocity=0 -> (none); origin xyz=0 0.1025 0.0306 rpy=1.5708 0 0 -> xyz=0 0.1025 0.0306 rpy=0 0 0
- joint Rotation: axis 0 1 0 -> 0 -1 0; limit lower=-2.1 upper=2.1 effort=0 velocity=0 -> (none)
- joint Wrist_Roll: axis 0 -1 0 -> 0 1 0; limit lower=-3.14159 upper=3.14159 effort=0 velocity=0 -> (none)
